File: hardware/MCU.kicad_sch (KiCad schematic)
At the start: 33 parts, among them SW1 reset, SW2 MCU_BOOT, U7 STM32H743VITx, Y1 ASE-8.000MHZ-LC-T

Commit message: hardware: import PCBWay manufacturing metadata variant
Parts:
- C21: Approved Distributor (none) -> DigiKey; DNP Status (none) -> POPULATE; Distributor Part Number (none) -> See sourcing URL; Lifecycle (none) -> Active; MPN (none) -> GRM188R71H103KA01D; Manufacturer (none) -> Murata; PCBWay Sourcing Note (none) -> PCBWay turnkey; exact MPN; Power Rating (none) -> N/A; Sourcing URL (none) -> https://www.digikey.com/en/products/result?keywords=GRM188R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; Substitution Policy (none) -> Equivalent only with written approval; Technology (none) -> X7R MLCC; Temperature Rating (none) -> -55..125 C; Tolerance (none) -> +/-10%; Voltage Rating (none) -> 50 V
- C22: Approved Distributor (none) -> DigiKey; DNP Status (none) -> POPULATE; Distributor Part Number (none) -> See sourcing URL; Lifecycle (none) -> Active; MPN (none) -> GRM188R61C475KE11D; Manufacturer (none) -> Murata; PCBWay Sourcing Note (none) -> PCBWay turnkey; exact MPN; Power Rating (none) -> N/A; Sourcing URL (none) -> https://www.digikey.com/en/products/result?keywords=GRM188R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; Substitution Policy (none) -> Equivalent only with written approval; Technology (none) -> X5R MLCC; Temperature Rating (none) -> -55..85 C; Tolerance (none) -> +/-10%; Voltage Rating (none) -> 16 V
- C23, C27: Approved Distributor (none) -> DigiKey; DNP Status (none) -> POPULATE; Distributor Part Number (none) -> See sourcing URL; Lifecycle (none) -> Active; MPN (none) -> GRM188R71C105KA12D; Manufacturer (none) -> Murata; PCBWay Sourcing Note (none) -> PCBWay turnkey; exact MPN; Power Rating (none) -> N/A; Sourcing URL (none) -> https://www.digikey.com/en/products/result?keywords=GRM188R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; Substitution Policy (none) -> Equivalent only with written approval; Technology (none) -> X7R MLCC; Temperature Rating (none) -> -55..125 C; Tolerance (none) -> +/-10%; Voltage Rating (none) -> 16 V
- C24, C25, C26, C28, C29, C31, C32: Approved Distributor (none) -> DigiKey; DNP Status (none) -> POPULATE; Distributor Part Number (none) -> See sourcing URL; Lifecycle (none) -> Active; MPN (none) -> GRM155R71H104KE14D; Manufacturer (none) -> Murata; PCBWay Sourcing Note (none) -> PCBWay turnkey; exact MPN; Power Rating (none) -> N/A; Sourcing URL (none) -> https://www.digikey.com/en/products/result?keywords=GRM155R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; Substitution Policy (none) -> Equivalent only with written approval; Technology (none) -> X7R MLCC; Temperature Rating (none) -> -55..125 C; Tolerance (none) -> +/-10%; Voltage Rating (none) -> 50 V
- C30: Approved Distributor (none) -> DigiKey; DNP Status (none) -> POPULATE; Distributor Part Number (none) -> See sourcing URL; Lifecycle (none) -> Active; MPN (none) -> GRM155R71H103KA88D; Manufacturer (none) -> Murata; PCBWay Sourcing Note (none) -> PCBWay turnkey; exact MPN; Power Rating (none) -> N/A; Sourcing URL (none) -> https://www.digikey.com/en/products/result?keywords=GRM155R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; Substitution Policy (none) -> Equivalent only with written approval; Technology (none) -> X7R MLCC; Temperature Rating (none) -> -55..125 C; Tolerance (none) -> +/-10%; Voltage Rating (none) -> 50 V
- C33: Approved Distributor (none) -> DigiKey; DNP Status (none) -> POPULATE; Distributor Part Number (none) -> See sourcing URL; Lifecycle (none) -> Active; MPN (none) -> GRM188R71H104KA93D; Manufacturer (none) -> Murata; PCBWay Sourcing Note (none) -> PCBWay turnkey; exact MPN; Power Rating (none) -> N/A; Sourcing URL (none) -> https://www.digikey.com/en/products/result?keywords=GRM188R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; Substitution Policy (none) -> Equivalent only with written approval; Technology (none) -> X7R MLCC; Temperature Rating (none) -> -55..125 C; Tolerance (none) -> +/-10%; Voltage Rating (none) -> 50 V
- C34, C35: Approved Distributor (none) -> DigiKey; DNP Status (none) -> POPULATE; Distributor Part Number (none) -> See sourcing URL; Lifecycle (none) -> Active; MPN (none) -> GRM188R71C225KE15D; Manufacturer (none) -> Murata; PCBWay Sourcing Note (none) -> PCBWay turnkey; exact MPN; Power Rating (none) -> N/A; Sourcing URL (none) -> https://www.digikey.com/en/products/result?keywords=GRM188R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; Substitution Policy (none) -> Equivalent only with written approval; Technology (none) -> X7R MLCC; Temperature Rating (none) -> -55..125 C; Tolerance (none) -> +/-10%; Voltage Rating (none) -> 16 V
- D6, D7: Approved Distributor (none) -> DigiKey; DNP Status (none) -> POPULATE; Distributor Part Number (none) -> See sourcing URL; Lifecycle (none) -> Active; MPN (none) -> LTST-C170KGKT; Manufacturer (none) -> Lite-On; PCBWay Sourcing Note (none) -> PCBWay turnkey; exact MPN; Power Rating (none) -> 75 mW; Sourcing URL (none) -> https://www.digikey.com/en/products/result?keywords=LTST-C1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; Substitution Policy (none) -> Equivalent only with written approval; Technology (none) -> InGaN LED; Temperature Rating (none) -> -55..85 C; Tolerance (none) -> N/A; Voltage Rating (none) -> 5 V rail
- FB1: Approved Distributor (none) -> DigiKey; DNP Status (none) -> POPULATE; Distributor Part Number (none) -> See sourcing URL; Lifecycle (none) -> Active; MPN (none) -> BLM18AG102SN1D; Manufacturer (none) -> Murata; PCBWay Sourcing Note (none) -> PCBWay turnkey; exact MPN; Power Rating (none) -> 500 mA; Sourcing URL (none) -> https://www.digikey.com/en/products/result?keywords=BLM18AG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; Substitution Policy (none) -> Equivalent only with written approval; Technology (none) -> Ferrite bead; Temperature Rating (none) -> -55..125 C; Tolerance (none) -> +/-25%; Voltage Rating (none) -> N/A
- R15, R16: Approved Distributor (none) -> DigiKey; DNP Status (none) -> POPULATE; Distributor Part Number (none) -> See sourcing URL; Lifecycle (none) -> Active; MPN (none) -> RC0402FR-0749R9L; Manufacturer (none) -> Yageo; PCBWay Sourcing Note (none) -> PCBWay turnkey; exact MPN; Power Rating (none) -> 0.0625 W; Sourcing URL (none) -> https://www.digikey.com/en/products/result?keywords=RC0402F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; Substitution Policy (none) -> Equivalent only with written approval; Technology (none) -> Thick-film resistor; Temperature Rating (none) -> -55..155 C; Tolerance (none) -> +/-1%; Voltage Rating (none) -> 50 V
- R17: Approved Distributor (none) -> DigiKey; DNP Status (none) -> POPULATE; Distributor Part Number (none) -> See sourcing URL; Lifecycle (none) -> Active; MPN (none) -> RC0402FR-07330RL; Manufacturer (none) -> Yageo; PCBWay Sourcing Note (none) -> PCBWay turnkey; exact MPN; Power Rating (none) -> 0.0625 W; Sourcing URL (none) -> https://www.digikey.com/en/products/result?keywords=RC0402F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; Substitution Policy (none) -> Equivalent only with written approval; Technology (none) -> Thick-film resistor; Temperature Rating (none) -> -55..155 C; Tolerance (none) -> +/-1%; Voltage Rating (none) -> 50 V
- R18: Approved Distributor (none) -> DigiKey; DNP Status (none) -> POPULATE; Distributor Part Number (none) -> See sourcing URL; Lifecycle (none) -> Active; MPN (none) -> RC0402FR-075K1L; Manufacturer (none) -> Yageo; PCBWay Sourcing Note (none) -> PCBWay turnkey; exact MPN; Power Rating (none) -> 0.0625 W; Sourcing URL (none) -> https://www.digikey.com/en/products/result?keywords=RC0402F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; Substitution Policy (none) -> Equivalent only with written approval; Technology (none) -> Thick-film resistor; Temperature Rating (none) -> -55..155 C; Tolerance (none) -> +/-1%; Voltage Rating (none) -> 50 V
- R6: Approved Distributor (none) -> DigiKey; DNP Status (none) -> POPULATE; Distributor Part Number (none) -> See sourcing URL; Lifecycle (none) -> Active; MPN (none) -> RC0402FR-075K23L; Manufacturer (none) -> Yageo; PCBWay Sourcing Note (none) -> PCBWay turnkey; exact MPN; Power Rating (none) -> 0.0625 W; Sourcing URL (none) -> https://www.digikey.com/en/products/result?keywords=RC0402F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; Substitution Policy (none) -> Equivalent only with written approval; Technology (none) -> Thick-film resistor; Temperature Rating (none) -> -55..155 C; Tolerance (none) -> +/-1%; Voltage Rating (none) -> 50 V
- R7: Approved Distributor (none) -> DigiKey; DNP Status (none) -> POPULATE; Distributor Part Number (none) -> See sourcing URL; Lifecycle (none) -> Active; MPN (none) -> RC0402FR-0720KL; Manufacturer (none) -> Yageo; PCBWay Sourcing Note (none) -> PCBWay turnkey; exact MPN; Power Rating (none) -> 0.0625 W; Sourcing URL (none) -> https://www.digikey.com/en/products/result?keywords=RC0402F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; Substitution Policy (none) -> Equivalent only with written approval; Technology (none) -> Thick-film resistor; Temperature Rating (none) -> -55..155 C; Tolerance (none) -> +/-1%; Voltage Rating (none) -> 50 V
- R8: Approved Distributor (none) -> DigiKey; DNP Status (none) -> POPULATE; Distributor Part Number (none) -> See sourcing URL; Lifecycle (none) -> Active; MPN (none) -> RC0402JR-070RL; Manufacturer (none) -> Yageo; PCBWay Sourcing Note (none) -> PCBWay turnkey; exact MPN; Power Rating (none) -> 0.0625 W; Sourcing URL (none) -> https://www.digikey.com/en/products/result?keywords=RC0402J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; Substitution Policy (none) -> Equivalent only with written approval; Technology (none) -> Thick-film resistor; Temperature Rating (none) -> -55..155 C; Tolerance (none) -> +/-5%; Voltage Rating (none) -> 50 V
- SW1, SW2: Approved Distributor (none) -> DigiKey; DNP Status (none) -> POPULATE; Distributor Part Number (none) -> 4809-SKRKAEE020TR-ND; Lifecycle (none) -> Active; MPN (none) -> SKRKAEE020; Manufacturer (none) -> Alps Alpine; PCBWay Sourcing Note (none) -> PCBWay turnkey; exact MPN; Power Rating (none) -> 50 mA; Sourcing URL (none) -> https://www.digikey.com/en/products/detail/alps-alpine/SKRK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; Substitution Policy (none) -> Equivalent only with written approval; Technology (none) -> Tact switch; Temperature Rating (none) -> -40..85 C; Tolerance (none) -> N/A; Voltage Rating (none) -> 12 V
- U7: value STM32H743VITx -> STM32H743VIT6; Approved Distributor (none) -> DigiKey; DNP Status (none) -> POPULATE; Distributor Part Number (none) -> See sourcing URL; Lifecycle (none) -> Active; MPN (none) -> STM32H743VIT6; Manufacturer (none) -> STMicroelectronics; PCBWay Sourcing Note (none) -> PCBWay turnkey; exact MPN; Power Rating (none) -> N/A; Sourcing URL (none) -> https://www.digikey.com/en/products/result?keywords=STM32H7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; Substitution Policy (none) -> NO SUBSTITUTE WITHOUT WRITTEN APPROVAL; Technology (none) -> Integrated circuit; Temperature Rating (none) -> -40..85 C minimum; Tolerance (none) -> N/A; Voltage Rating (none) -> Per datasheet
- Y1: value ASE-8.000MHZ-LC-T -> ASE-8.000MHZ-L-C-T; Approved Distributor (none) -> DigiKey; DNP Status (none) -> POPULATE; Distributor Part Number (none) -> 535-ASE-8.000MHZ-L-C-TTR-ND; Lifecycle (none) -> Active; MPN (none) -> ASE-8.000MHZ-L-C-T; Manufacturer (none) -> Abracon; PCBWay Sourcing Note (none) -> PCBWay turnkey; exact MPN; Power Rating (none) -> N/A; Sourcing URL (none) -> https://www.digikey.com/en/products/detail/abracon-llc/ASE-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; Substitution Policy (none) -> NO SUBSTITUTE WITHOUT WRITTEN APPROVAL; Technology (none) -> CMOS oscillator; Temperature Rating (none) -> -40..85 C; Tolerance (none) -> +/-25 ppm; Voltage Rating (none) -> 3.3 V
