File: hardware/Sensors.kicad_sch (KiCad schematic)
At the start: 43 parts, among them U10 BMI270, U11 LIS3MDLTR, U12 BMP388, U13 AT7456E, U14 SN65HVD230, U8 ICM-42688-P, U9 W25Q128JVSIQ, Y2 27Mhz 20pF

Commit message: hardware: import PCBWay manufacturing metadata variant
Parts:
- C36, C37, C43, C44, C46, C50, C51, C52, C53, C54, C55: Approved Distributor (none) -> DigiKey; DNP Status (none) -> POPULATE; Distributor Part Number (none) -> See sourcing URL; Lifecycle (none) -> Active; MPN (none) -> GRM155R71H104KE14D; Manufacturer (none) -> Murata; PCBWay Sourcing Note (none) -> PCBWay turnkey; exact MPN; Power Rating (none) -> N/A; Sourcing URL (none) -> https://www.digikey.com/en/products/result?keywords=GRM155R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; Substitution Policy (none) -> Equivalent only with written approval; Technology (none) -> X7R MLCC; Temperature Rating (none) -> -55..125 C; Tolerance (none) -> +/-10%; Voltage Rating (none) -> 50 V
- C38: Approved Distributor (none) -> DigiKey; DNP Status (none) -> POPULATE; Distributor Part Number (none) -> See sourcing URL; Lifecycle (none) -> Active; MPN (none) -> GRM188R71C225KE15D; Manufacturer (none) -> Murata; PCBWay Sourcing Note (none) -> PCBWay turnkey; exact MPN; Power Rating (none) -> N/A; Sourcing URL (none) -> https://www.digikey.com/en/products/result?keywords=GRM188R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; Substitution Policy (none) -> Equivalent only with written approval; Technology (none) -> X7R MLCC; Temperature Rating (none) -> -55..125 C; Tolerance (none) -> +/-10%; Voltage Rating (none) -> 16 V
- C39: Approved Distributor (none) -> DigiKey; DNP Status (none) -> POPULATE; Distributor Part Number (none) -> See sourcing URL; Lifecycle (none) -> Active; MPN (none) -> GRM155R71H103KA88D; Manufacturer (none) -> Murata; PCBWay Sourcing Note (none) -> PCBWay turnkey; exact MPN; Power Rating (none) -> N/A; Sourcing URL (none) -> https://www.digikey.com/en/products/result?keywords=GRM155R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; Substitution Policy (none) -> Equivalent only with written approval; Technology (none) -> X7R MLCC; Temperature Rating (none) -> -55..125 C; Tolerance (none) -> +/-10%; Voltage Rating (none) -> 50 V
- C45, C47: Approved Distributor (none) -> DigiKey; DNP Status (none) -> POPULATE; Distributor Part Number (none) -> See sourcing URL; Lifecycle (none) -> Active; MPN (none) -> GRM1555C1H300JA01D; Manufacturer (none) -> Murata; PCBWay Sourcing Note (none) -> PCBWay turnkey; exact MPN; Power Rating (none) -> N/A; Sourcing URL (none) -> https://www.digikey.com/en/products/result?keywords=GRM1555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; Substitution Policy (none) -> Equivalent only with written approval; Technology (none) -> C0G/NP0 MLCC; Temperature Rating (none) -> -55..125 C; Tolerance (none) -> +/-5%; Voltage Rating (none) -> 50 V
- C48, C49: Approved Distributor (none) -> DigiKey; DNP Status (none) -> POPULATE; Distributor Part Number (none) -> See sourcing URL; Lifecycle (none) -> Active; MPN (none) -> GRM188C61E226ME01D; Manufacturer (none) -> Murata; PCBWay Sourcing Note (none) -> PCBWay turnkey; exact MPN; Power Rating (none) -> N/A; Sourcing URL (none) -> https://www.digikey.com/en/products/detail/murata-electroni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; Substitution Policy (none) -> Equivalent only with written approval and DC-bias review; Technology (none) -> X5S MLCC; Temperature Rating (none) -> -55..85 C; Tolerance (none) -> +/-20%; Voltage Rating (none) -> 25 V
- D8: Approved Distributor (none) -> DigiKey; DNP Status (none) -> POPULATE; Distributor Part Number (none) -> See sourcing URL; Lifecycle (none) -> Active; MPN (none) -> SM712-02HTG; Manufacturer (none) -> Littelfuse; PCBWay Sourcing Note (none) -> PCBWay turnkey; exact MPN; Power Rating (none) -> 600 W pulse; Sourcing URL (none) -> https://www.digikey.com/en/products/result?keywords=SM712-0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; Substitution Policy (none) -> NO SUBSTITUTE without written approval; Technology (none) -> TVS array; Temperature Rating (none) -> -40..125 C; Tolerance (none) -> N/A; Voltage Rating (none) -> 12/-7 V standoff
- R19, R22: Approved Distributor (none) -> DigiKey; DNP Status (none) -> POPULATE; Distributor Part Number (none) -> See sourcing URL; Lifecycle (none) -> Active; MPN (none) -> RC0402FR-07330RL; Manufacturer (none) -> Yageo; PCBWay Sourcing Note (none) -> PCBWay turnkey; exact MPN; Power Rating (none) -> 0.0625 W; Sourcing URL (none) -> https://www.digikey.com/en/products/result?keywords=RC0402F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; Substitution Policy (none) -> Equivalent only with written approval; Technology (none) -> Thick-film resistor; Temperature Rating (none) -> -55..155 C; Tolerance (none) -> +/-1%; Voltage Rating (none) -> 50 V
- R20, R21: Approved Distributor (none) -> DigiKey; DNP Status (none) -> POPULATE; Distributor Part Number (none) -> See sourcing URL; Lifecycle (none) -> Active; MPN (none) -> RC0402FR-0710KL; Manufacturer (none) -> Yageo; PCBWay Sourcing Note (none) -> PCBWay turnkey; exact MPN; Power Rating (none) -> 0.0625 W; Sourcing URL (none) -> https://www.digikey.com/en/products/result?keywords=RC0402F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; Substitution Policy (none) -> Equivalent only with written approval; Technology (none) -> Thick-film resistor; Temperature Rating (none) -> -55..155 C; Tolerance (none) -> +/-1%; Voltage Rating (none) -> 50 V
- R23, R24: Approved Distributor (none) -> DigiKey; DNP Status (none) -> POPULATE; Distributor Part Number (none) -> See sourcing URL; Lifecycle (none) -> Active; MPN (none) -> RC0402JR-070RL; Manufacturer (none) -> Yageo; PCBWay Sourcing Note (none) -> PCBWay turnkey; exact MPN; Power Rating (none) -> 0.0625 W; Sourcing URL (none) -> https://www.digikey.com/en/products/result?keywords=RC0402J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; Substitution Policy (none) -> Equivalent only with written approval; Technology (none) -> Thick-film resistor; Temperature Rating (none) -> -55..155 C; Tolerance (none) -> +/-5%; Voltage Rating (none) -> 50 V
- R25, R26, R31, R32: Approved Distributor (none) -> DigiKey; DNP Status (none) -> POPULATE; Distributor Part Number (none) -> See sourcing URL; Lifecycle (none) -> Active; MPN (none) -> RC0402FR-074K7L; Manufacturer (none) -> Yageo; PCBWay Sourcing Note (none) -> PCBWay turnkey; exact MPN; Power Rating (none) -> 0.0625 W; Sourcing URL (none) -> https://www.digikey.com/en/products/result?keywords=RC0402F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; Substitution Policy (none) -> Equivalent only with written approval; Technology (none) -> Thick-film resistor; Temperature Rating (none) -> -55..155 C; Tolerance (none) -> +/-1%; Voltage Rating (none) -> 50 V
- R27, R28: Approved Distributor (none) -> DigiKey; DNP Status (none) -> POPULATE; Distributor Part Number (none) -> See sourcing URL; Lifecycle (none) -> Active; MPN (none) -> RC0402FR-0775RL; Manufacturer (none) -> Yageo; PCBWay Sourcing Note (none) -> PCBWay turnkey; exact MPN; Power Rating (none) -> 0.0625 W; Sourcing URL (none) -> https://www.digikey.com/en/products/result?keywords=RC0402F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; Substitution Policy (none) -> Equivalent only with written approval; Technology (none) -> Thick-film resistor; Temperature Rating (none) -> -55..155 C; Tolerance (none) -> +/-1%; Voltage Rating (none) -> 50 V
- R29, R30: Approved Distributor (none) -> DigiKey; DNP Status (none) -> POPULATE; Distributor Part Number (none) -> See sourcing URL; Lifecycle (none) -> Active; MPN (none) -> RC0402FR-077K5L; Manufacturer (none) -> Yageo; PCBWay Sourcing Note (none) -> PCBWay turnkey; exact MPN; Power Rating (none) -> 0.0625 W; Sourcing URL (none) -> https://www.digikey.com/en/products/result?keywords=RC0402F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; Substitution Policy (none) -> Equivalent only with written approval; Technology (none) -> Thick-film resistor; Temperature Rating (none) -> -55..155 C; Tolerance (none) -> +/-1%; Voltage Rating (none) -> 50 V
- U10: Approved Distributor (none) -> DigiKey; DNP Status (none) -> POPULATE; Distributor Part Number (none) -> See sourcing URL; Lifecycle (none) -> Active; MPN (none) -> BMI270; Manufacturer (none) -> Bosch Sensortec; PCBWay Sourcing Note (none) -> PCBWay turnkey; exact MPN; Power Rating (none) -> N/A; Sourcing URL (none) -> https://www.digikey.com/en/products/result?keywords=BMI270; Substitution Policy (none) -> NO SUBSTITUTE WITHOUT WRITTEN APPROVAL; Technology (none) -> Integrated circuit; Temperature Rating (none) -> -40..85 C minimum; Tolerance (none) -> N/A; Voltage Rating (none) -> Per datasheet
- U12: Approved Distributor (none) -> DigiKey; DNP Status (none) -> POPULATE; Distributor Part Number (none) -> See sourcing URL; Lifecycle (none) -> Active; MPN (none) -> BMP388; Manufacturer (none) -> Bosch Sensortec; PCBWay Sourcing Note (none) -> PCBWay turnkey; exact MPN; Power Rating (none) -> N/A; Sourcing URL (none) -> https://www.digikey.com/en/products/result?keywords=BMP388; Substitution Policy (none) -> NO SUBSTITUTE WITHOUT WRITTEN APPROVAL; Technology (none) -> Integrated circuit; Temperature Rating (none) -> -40..85 C minimum; Tolerance (none) -> N/A; Voltage Rating (none) -> Per datasheet
- U13: Approved Distributor (none) -> LCSC; DNP Status (none) -> POPULATE; Distributor Part Number (none) -> C82351; Lifecycle (none) -> Active; MPN (none) -> AT7456E; Manufacturer (none) -> ZHONGKEWEI; PCBWay Sourcing Note (none) -> PCBWay turnkey; exact MPN; Power Rating (none) -> N/A; Sourcing URL (none) -> https://www.lcsc.com/product-detail/C82351.html; Substitution Policy (none) -> NO SUBSTITUTE WITHOUT WRITTEN APPROVAL; Technology (none) -> Integrated circuit; Temperature Rating (none) -> -40..85 C minimum; Tolerance (none) -> N/A; Voltage Rating (none) -> Per datasheet
- U14: Approved Distributor (none) -> DigiKey; DNP Status (none) -> POPULATE; Distributor Part Number (none) -> See sourcing URL; Lifecycle (none) -> Active; MPN (none) -> SN65HVD230DR; Manufacturer (none) -> Texas Instruments; PCBWay Sourcing Note (none) -> PCBWay turnkey; exact MPN; Power Rating (none) -> N/A; Sourcing URL (none) -> https://www.digikey.com/en/products/result?keywords=SN65HVD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; Substitution Policy (none) -> NO SUBSTITUTE WITHOUT WRITTEN APPROVAL; Technology (none) -> Integrated circuit; Temperature Rating (none) -> -40..85 C minimum; Tolerance (none) -> N/A; Voltage Rating (none) -> Per datasheet
- U8: Approved Distributor (none) -> DigiKey; DNP Status (none) -> POPULATE; Distributor Part Number (none) -> See sourcing URL; Lifecycle (none) -> Active; MPN (none) -> ICM-42688-P; Manufacturer (none) -> TDK InvenSense; PCBWay Sourcing Note (none) -> PCBWay turnkey; exact MPN; Power Rating (none) -> N/A; Sourcing URL (none) -> https://www.digikey.com/en/products/result?keywords=ICM-426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; Substitution Policy (none) -> NO SUBSTITUTE WITHOUT WRITTEN APPROVAL; Technology (none) -> Integrated circuit; Temperature Rating (none) -> -40..85 C minimum; Tolerance (none) -> N/A; Voltage Rating (none) -> Per datasheet
- U9: Approved Distributor (none) -> DigiKey; DNP Status (none) -> POPULATE; Distributor Part Number (none) -> See sourcing URL; Lifecycle (none) -> Active; MPN (none) -> W25Q128JVSIQ; Manufacturer (none) -> Winbond; PCBWay Sourcing Note (none) -> PCBWay turnkey; exact MPN; Power Rating (none) -> N/A; Sourcing URL (none) -> https://www.digikey.com/en/products/result?keywords=W25Q128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; Substitution Policy (none) -> NO SUBSTITUTE WITHOUT WRITTEN APPROVAL; Technology (none) -> Integrated circuit; Temperature Rating (none) -> -40..85 C minimum; Tolerance (none) -> N/A; Voltage Rating (none) -> Per datasheet
- Y2: value 27Mhz 20pF -> TSX-3225 27.00M-N0AANNG40RG3; Approved Distributor (none) -> DigiKey; DNP Status (none) -> POPULATE; Distributor Part Number (none) -> 114-TSX-322527.00M-N0AANNG40RG3TR-ND; Lifecycle (none) -> Active; MPN (none) -> TSX-3225 27.00M-N0AANNG40RG3; Manufacturer (none) -> Epson; PCBWay Sourcing Note (none) -> PCBWay turnkey; exact MPN; Power Rating (none) -> 100 uW drive; Sourcing URL (none) -> https://www.digikey.com/en/products/detail/epson/TSX-3225-2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; Substitution Policy (none) -> NO SUBSTITUTE WITHOUT WRITTEN APPROVAL; Technology (none) -> Quartz crystal; Temperature Rating (none) -> -40..85 C; Tolerance (none) -> +/-10 ppm; Voltage Rating (none) -> N/A
