File: hardware/connectors.kicad_sch (KiCad schematic)
At the start: 53 parts, among them J10 CAN BUS, J11 MAVLINK SIGNAL-ONLY, J12 POWER1 REGULATED 5.2V IN, J2 FPV, J3 ST_LINK, J4 GPS, J5 Airspeed sensor, J6 OpenESC SIGNAL-ONLY, J7 RC Receiver, J8 VTX, J9 DJI

Commit message: hardware: import PCBWay manufacturing metadata variant
Parts:
- J10, J11, J2, J3, J5, J7, J8: Approved Distributor (none) -> DigiKey; DNP Status (none) -> POPULATE; Distributor Part Number (none) -> See sourcing URL; Lifecycle (none) -> Active; MPN (none) -> SM04B-SRSS-TB(LF)(SN); Manufacturer (none) -> JST; PCBWay Sourcing Note (none) -> PCBWay turnkey; exact MPN; Power Rating (none) -> 1 A/contact; Sourcing URL (none) -> https://www.digikey.com/en/products/result?keywords=SM04B-S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; Substitution Policy (none) -> NO SUBSTITUTE without written approval; Technology (none) -> Connector; Temperature Rating (none) -> -25..85 C; Tolerance (none) -> N/A; Voltage Rating (none) -> 50 V
- J12: Approved Distributor (none) -> DigiKey; DNP Status (none) -> POPULATE; Distributor Part Number (none) -> WM15082-ND; Lifecycle (none) -> Active; PCBWay Sourcing Note (none) -> PCBWay THT; exact black/gold MPN only; Power Rating (none) -> 8 A/contact per vendor conditions; Sourcing URL (none) -> https://www.digikey.com/en/products/detail/molex/1053111202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; Substitution Policy (none) -> NO SUBSTITUTE WITHOUT WRITTEN APPROVAL; Technology (none) -> Connector; Temperature Rating (none) -> -40..105 C; Tolerance (none) -> N/A; Voltage Rating (none) -> 250 V
- J4, J9: Approved Distributor (none) -> DigiKey; DNP Status (none) -> POPULATE; Distributor Part Number (none) -> See sourcing URL; Lifecycle (none) -> Active; MPN (none) -> SM06B-SRSS-TB(LF)(SN); Manufacturer (none) -> JST; PCBWay Sourcing Note (none) -> PCBWay turnkey; exact MPN; Power Rating (none) -> 1 A/contact; Sourcing URL (none) -> https://www.digikey.com/en/products/result?keywords=SM06B-S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; Substitution Policy (none) -> NO SUBSTITUTE without written approval; Technology (none) -> Connector; Temperature Rating (none) -> -25..85 C; Tolerance (none) -> N/A; Voltage Rating (none) -> 50 V
- J6: Approved Distributor (none) -> DigiKey; DNP Status (none) -> POPULATE; Distributor Part Number (none) -> See sourcing URL; Lifecycle (none) -> Active; MPN (none) -> SM08B-SRSS-TB(LF)(SN); Manufacturer (none) -> JST; PCBWay Sourcing Note (none) -> PCBWay turnkey; exact MPN; Power Rating (none) -> 1 A/contact; Sourcing URL (none) -> https://www.digikey.com/en/products/result?keywords=SM08B-S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; Substitution Policy (none) -> NO SUBSTITUTE without written approval; Technology (none) -> Connector; Temperature Rating (none) -> -25..85 C; Tolerance (none) -> N/A; Voltage Rating (none) -> 50 V
