File: hardware/power.kicad_sch (KiCad schematic)
At the start: 44 parts, among them J1 USB4110GFA, Q1 AO3407A, U1 TPS54302, U2 USBLC6-2SC6, U3 INA226, U5 AP2112K-3.3, U6 AP7343-33W5-7

Commit message: hardware: import PCBWay manufacturing metadata variant
Parts:
- C1, C10, C3: Approved Distributor (none) -> DigiKey; DNP Status (none) -> POPULATE; Distributor Part Number (none) -> See sourcing URL; Lifecycle (none) -> Active; MPN (none) -> GRM188R6YA106MA73D; Manufacturer (none) -> Murata; PCBWay Sourcing Note (none) -> PCBWay turnkey; exact MPN; Power Rating (none) -> N/A; Sourcing URL (none) -> https://www.digikey.com/en/products/detail/murata-electroni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; Substitution Policy (none) -> NO SUBSTITUTE without written approval; verify 6S DC-bias d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; Technology (none) -> X5R MLCC; Temperature Rating (none) -> -55..85 C; Tolerance (none) -> +/-20%; Voltage Rating (none) -> 35 V
- C15, C16, C6, C7: Approved Distributor (none) -> DigiKey; DNP Status (none) -> POPULATE; Distributor Part Number (none) -> See sourcing URL; Lifecycle (none) -> Active; MPN (none) -> GRM188C61E226ME01D; Manufacturer (none) -> Murata; PCBWay Sourcing Note (none) -> PCBWay turnkey; exact MPN; Power Rating (none) -> N/A; Sourcing URL (none) -> https://www.digikey.com/en/products/detail/murata-electroni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; Substitution Policy (none) -> Equivalent only with written approval and DC-bias review; Technology (none) -> X5S MLCC; Temperature Rating (none) -> -55..85 C; Tolerance (none) -> +/-20%; Voltage Rating (none) -> 25 V
- C17, C18, C20: Approved Distributor (none) -> DigiKey; DNP Status (none) -> POPULATE; Distributor Part Number (none) -> See sourcing URL; Lifecycle (none) -> Active; MPN (none) -> GRM188R71C105KA12D; Manufacturer (none) -> Murata; PCBWay Sourcing Note (none) -> PCBWay turnkey; exact MPN; Power Rating (none) -> N/A; Sourcing URL (none) -> https://www.digikey.com/en/products/result?keywords=GRM188R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; Substitution Policy (none) -> Equivalent only with written approval; Technology (none) -> X7R MLCC; Temperature Rating (none) -> -55..125 C; Tolerance (none) -> +/-10%; Voltage Rating (none) -> 16 V
- C19: Approved Distributor (none) -> DigiKey; DNP Status (none) -> POPULATE; Distributor Part Number (none) -> See sourcing URL; Lifecycle (none) -> Active; MPN (none) -> GRM188R61C475KE11D; Manufacturer (none) -> Murata; PCBWay Sourcing Note (none) -> PCBWay turnkey; exact MPN; Power Rating (none) -> N/A; Sourcing URL (none) -> https://www.digikey.com/en/products/result?keywords=GRM188R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; Substitution Policy (none) -> Equivalent only with written approval; Technology (none) -> X5R MLCC; Temperature Rating (none) -> -55..85 C; Tolerance (none) -> +/-10%; Voltage Rating (none) -> 16 V
- C2, C5: Approved Distributor (none) -> DigiKey; DNP Status (none) -> POPULATE; Distributor Part Number (none) -> See sourcing URL; Lifecycle (none) -> Active; MPN (none) -> GRM155R71H104KE14D; Manufacturer (none) -> Murata; PCBWay Sourcing Note (none) -> PCBWay turnkey; exact MPN; Power Rating (none) -> N/A; Sourcing URL (none) -> https://www.digikey.com/en/products/result?keywords=GRM155R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; Substitution Policy (none) -> Equivalent only with written approval; Technology (none) -> X7R MLCC; Temperature Rating (none) -> -55..125 C; Tolerance (none) -> +/-10%; Voltage Rating (none) -> 50 V
- C4: Approved Distributor (none) -> DigiKey; DNP Status (none) -> POPULATE; Distributor Part Number (none) -> See sourcing URL; Lifecycle (none) -> Active; MPN (none) -> C2012X5R1V226M125AC; Manufacturer (none) -> TDK; PCBWay Sourcing Note (none) -> PCBWay exact-MPN quotation; Power Rating (none) -> N/A; Sourcing URL (none) -> https://www.digikey.com/en/products/result?keywords=C2012X5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; Substitution Policy (none) -> NO SUBSTITUTE without written approval; verify 6S DC-bias d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; Technology (none) -> X5R MLCC; Temperature Rating (none) -> -55..85 C; Tolerance (none) -> +/-20%; Voltage Rating (none) -> 35 V
- C8: Approved Distributor (none) -> DigiKey; DNP Status (none) -> POPULATE; Distributor Part Number (none) -> See sourcing URL; Lifecycle (none) -> Active; MPN (none) -> GRM1555C1H750JA01D; Manufacturer (none) -> Murata; PCBWay Sourcing Note (none) -> PCBWay turnkey; exact MPN; Power Rating (none) -> N/A; Sourcing URL (none) -> https://www.digikey.com/en/products/result?keywords=GRM1555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; Substitution Policy (none) -> Equivalent only with written approval; Technology (none) -> C0G/NP0 MLCC; Temperature Rating (none) -> -55..125 C; Tolerance (none) -> +/-5%; Voltage Rating (none) -> 50 V
- C9: Approved Distributor (none) -> DigiKey; DNP Status (none) -> POPULATE; Distributor Part Number (none) -> See sourcing URL; Lifecycle (none) -> Active; MPN (none) -> GRM155R61A475MEAAD; Manufacturer (none) -> Murata; PCBWay Sourcing Note (none) -> PCBWay turnkey; exact MPN; Power Rating (none) -> N/A; Sourcing URL (none) -> https://www.digikey.com/en/products/result?keywords=GRM155R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; Substitution Policy (none) -> Equivalent only with written approval; Technology (none) -> X5R MLCC; Temperature Rating (none) -> -55..85 C; Tolerance (none) -> +/-20%; Voltage Rating (none) -> 10 V
- D1: Approved Distributor (none) -> DigiKey; DNP Status (none) -> POPULATE; Distributor Part Number (none) -> See sourcing URL; Lifecycle (none) -> Active; MPN (none) -> SMF26A-E3-08; Manufacturer (none) -> Vishay; PCBWay Sourcing Note (none) -> PCBWay turnkey; exact MPN; Power Rating (none) -> 200 W pulse; Sourcing URL (none) -> https://www.digikey.com/en/products/result?keywords=SMF26A-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; Substitution Policy (none) -> NO SUBSTITUTE without written approval; Technology (none) -> TVS diode; Temperature Rating (none) -> -55..150 C; Tolerance (none) -> N/A; Voltage Rating (none) -> 26 V standoff
- D2: Approved Distributor (none) -> DigiKey; DNP Status (none) -> POPULATE; Distributor Part Number (none) -> See sourcing URL; Lifecycle (none) -> Active; MPN (none) -> BZT52C12-13-F; Manufacturer (none) -> Diodes Incorporated; PCBWay Sourcing Note (none) -> PCBWay turnkey; exact MPN; Power Rating (none) -> 500 mW; Sourcing URL (none) -> https://www.digikey.com/en/products/result?keywords=BZT52C1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; Substitution Policy (none) -> Equivalent only with written approval; Technology (none) -> Zener diode; Temperature Rating (none) -> -65..150 C; Tolerance (none) -> +/-5%; Voltage Rating (none) -> 12 V
- D4, D5: Approved Distributor (none) -> DigiKey; DNP Status (none) -> POPULATE; Distributor Part Number (none) -> See sourcing URL; Lifecycle (none) -> Active; MPN (none) -> LTST-C170KGKT; Manufacturer (none) -> Lite-On; PCBWay Sourcing Note (none) -> PCBWay turnkey; exact MPN; Power Rating (none) -> 75 mW; Sourcing URL (none) -> https://www.digikey.com/en/products/result?keywords=LTST-C1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; Substitution Policy (none) -> Equivalent only with written approval; Technology (none) -> InGaN LED; Temperature Rating (none) -> -55..85 C; Tolerance (none) -> N/A; Voltage Rating (none) -> 5 V rail
- J1: Approved Distributor (none) -> DigiKey; DNP Status (none) -> POPULATE; Distributor Part Number (none) -> See sourcing URL; Lifecycle (none) -> Active; MPN (none) -> USB4110-GF-A; Manufacturer (none) -> GCT; PCBWay Sourcing Note (none) -> PCBWay turnkey; exact MPN; Power Rating (none) -> N/A; Sourcing URL (none) -> https://www.digikey.com/en/products/detail/gct/USB4110-GF-A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; Substitution Policy (none) -> NO SUBSTITUTE without written approval; Technology (none) -> Connector; Temperature Rating (none) -> -40..85 C; Tolerance (none) -> N/A; Voltage Rating (none) -> 20 V
- L1: Approved Distributor (none) -> Coilcraft / Mouser; DNP Status (none) -> POPULATE; Distributor Part Number (none) -> See sourcing URL; Lifecycle (none) -> Active; MPN (none) -> XAL5050-153MEB; Manufacturer (none) -> Coilcraft; PCBWay Sourcing Note (none) -> PCBWay turnkey; exact MPN; Power Rating (none) -> Irms 3.7 A; Isat 3.9 A; Sourcing URL (none) -> https://www.coilcraft.com/en-us/products/power/shielded-ind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; Substitution Policy (none) -> NO SUBSTITUTE without written approval; Technology (none) -> Shielded molded inductor; Temperature Rating (none) -> -40..125 C; Tolerance (none) -> +/-20%; Voltage Rating (none) -> N/A
- Q1: Approved Distributor (none) -> DigiKey; DNP Status (none) -> POPULATE; Distributor Part Number (none) -> See sourcing URL; Lifecycle (none) -> Active; MPN (none) -> AO3407A; Manufacturer (none) -> Alpha & Omega Semiconductor; PCBWay Sourcing Note (none) -> PCBWay turnkey; exact MPN; Power Rating (none) -> 1.4 W; Sourcing URL (none) -> https://www.digikey.com/en/products/result?keywords=AO3407A; Substitution Policy (none) -> NO SUBSTITUTE without written approval; Technology (none) -> P-channel MOSFET; Temperature Rating (none) -> -55..150 C; Tolerance (none) -> N/A; Voltage Rating (none) -> 30 V
- R1: Approved Distributor (none) -> DigiKey; DNP Status (none) -> POPULATE; Distributor Part Number (none) -> See sourcing URL; Lifecycle (none) -> Active; MPN (none) -> RC0402FR-075K1L; Manufacturer (none) -> Yageo; PCBWay Sourcing Note (none) -> PCBWay turnkey; exact MPN; Power Rating (none) -> 0.0625 W; Sourcing URL (none) -> https://www.digikey.com/en/products/result?keywords=RC0402F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; Substitution Policy (none) -> Equivalent only with written approval; Technology (none) -> Thick-film resistor; Temperature Rating (none) -> -55..155 C; Tolerance (none) -> +/-1%; Voltage Rating (none) -> 50 V
- R10: Approved Distributor (none) -> DigiKey; DNP Status (none) -> POPULATE; Distributor Part Number (none) -> See sourcing URL; Lifecycle (none) -> Active; MPN (none) -> RC0402FR-07330RL; Manufacturer (none) -> Yageo; PCBWay Sourcing Note (none) -> PCBWay turnkey; exact MPN; Power Rating (none) -> 0.0625 W; Sourcing URL (none) -> https://www.digikey.com/en/products/result?keywords=RC0402F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; Substitution Policy (none) -> Equivalent only with written approval; Technology (none) -> Thick-film resistor; Temperature Rating (none) -> -55..155 C; Tolerance (none) -> +/-1%; Voltage Rating (none) -> 50 V
- R11, R2: Approved Distributor (none) -> DigiKey; DNP Status (none) -> POPULATE; Distributor Part Number (none) -> See sourcing URL; Lifecycle (none) -> Active; MPN (none) -> RC0402FR-07100KL; Manufacturer (none) -> Yageo; PCBWay Sourcing Note (none) -> PCBWay turnkey; exact MPN; Power Rating (none) -> 0.0625 W; Sourcing URL (none) -> https://www.digikey.com/en/products/result?keywords=RC0402F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; Substitution Policy (none) -> Equivalent only with written approval; Technology (none) -> Thick-film resistor; Temperature Rating (none) -> -55..155 C; Tolerance (none) -> +/-1%; Voltage Rating (none) -> 50 V
- R12, R13, R14: Approved Distributor (none) -> DigiKey; DNP Status (none) -> POPULATE; Distributor Part Number (none) -> See sourcing URL; Lifecycle (none) -> Active; MPN (none) -> RC0402FR-0710KL; Manufacturer (none) -> Yageo; PCBWay Sourcing Note (none) -> PCBWay turnkey; exact MPN; Power Rating (none) -> 0.0625 W; Sourcing URL (none) -> https://www.digikey.com/en/products/result?keywords=RC0402F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; Substitution Policy (none) -> Equivalent only with written approval; Technology (none) -> Thick-film resistor; Temperature Rating (none) -> -55..155 C; Tolerance (none) -> +/-1%; Voltage Rating (none) -> 50 V
- R3, R4: Approved Distributor (none) -> DigiKey; DNP Status (none) -> POPULATE; Distributor Part Number (none) -> See sourcing URL; Lifecycle (none) -> Active; MPN (none) -> RC0402FR-0749R9L; Manufacturer (none) -> Yageo; PCBWay Sourcing Note (none) -> PCBWay turnkey; exact MPN; Power Rating (none) -> 0.0625 W; Sourcing URL (none) -> https://www.digikey.com/en/products/result?keywords=RC0402F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; Substitution Policy (none) -> Equivalent only with written approval; Technology (none) -> Thick-film resistor; Temperature Rating (none) -> -55..155 C; Tolerance (none) -> +/-1%; Voltage Rating (none) -> 50 V
- R5, R5B1: Approved Distributor (none) -> DigiKey; DNP Status (none) -> POPULATE; Distributor Part Number (none) -> See sourcing URL; Lifecycle (none) -> Active; MPN (none) -> RC0402FR-077K15L; Manufacturer (none) -> Yageo; PCBWay Sourcing Note (none) -> PCBWay turnkey; exact MPN; Power Rating (none) -> 0.0625 W; Sourcing URL (none) -> https://www.digikey.com/en/products/result?keywords=RC0402F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; Substitution Policy (none) -> Equivalent only with written approval; Technology (none) -> Thick-film resistor; Temperature Rating (none) -> -55..155 C; Tolerance (none) -> +/-1%; Voltage Rating (none) -> 50 V
- R5C1: Approved Distributor (none) -> DigiKey; DNP Status (none) -> POPULATE; Distributor Part Number (none) -> See sourcing URL; Lifecycle (none) -> Active; MPN (none) -> RC0402FR-075K23L; Manufacturer (none) -> Yageo; PCBWay Sourcing Note (none) -> PCBWay turnkey; exact MPN; Power Rating (none) -> 0.0625 W; Sourcing URL (none) -> https://www.digikey.com/en/products/result?keywords=RC0402F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; Substitution Policy (none) -> Equivalent only with written approval; Technology (none) -> Thick-film resistor; Temperature Rating (none) -> -55..155 C; Tolerance (none) -> +/-1%; Voltage Rating (none) -> 50 V
- U1: Approved Distributor (none) -> DigiKey; DNP Status (none) -> POPULATE; Distributor Part Number (none) -> See sourcing URL; Lifecycle (none) -> Active; MPN (none) -> TPS54302DDCR; Manufacturer (none) -> Texas Instruments; PCBWay Sourcing Note (none) -> PCBWay turnkey; exact MPN; Power Rating (none) -> N/A; Sourcing URL (none) -> https://www.digikey.com/en/products/result?keywords=TPS5430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; Substitution Policy (none) -> NO SUBSTITUTE WITHOUT WRITTEN APPROVAL; Technology (none) -> Integrated circuit; Temperature Rating (none) -> -40..85 C minimum; Tolerance (none) -> N/A; Voltage Rating (none) -> Per datasheet
- U2: Approved Distributor (none) -> DigiKey; DNP Status (none) -> POPULATE; Distributor Part Number (none) -> See sourcing URL; Lifecycle (none) -> Active; MPN (none) -> USBLC6-2SC6; Manufacturer (none) -> STMicroelectronics; PCBWay Sourcing Note (none) -> PCBWay turnkey; exact MPN; Power Rating (none) -> N/A; Sourcing URL (none) -> https://www.digikey.com/en/products/result?keywords=USBLC6-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; Substitution Policy (none) -> NO SUBSTITUTE WITHOUT WRITTEN APPROVAL; Technology (none) -> Integrated circuit; Temperature Rating (none) -> -40..85 C minimum; Tolerance (none) -> N/A; Voltage Rating (none) -> Per datasheet
- U5: Approved Distributor (none) -> DigiKey; DNP Status (none) -> POPULATE; Distributor Part Number (none) -> See sourcing URL; Lifecycle (none) -> Active; MPN (none) -> AP2112K-3.3TRG1; Manufacturer (none) -> Diodes Incorporated; PCBWay Sourcing Note (none) -> PCBWay turnkey; exact MPN; Power Rating (none) -> N/A; Sourcing URL (none) -> https://www.digikey.com/en/products/result?keywords=AP2112K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; Substitution Policy (none) -> NO SUBSTITUTE WITHOUT WRITTEN APPROVAL; Technology (none) -> Integrated circuit; Temperature Rating (none) -> -40..85 C minimum; Tolerance (none) -> N/A; Voltage Rating (none) -> Per datasheet
- U6: Approved Distributor (none) -> DigiKey; DNP Status (none) -> POPULATE; Distributor Part Number (none) -> See sourcing URL; Lifecycle (none) -> Active; MPN (none) -> AP7343-33W5-7; Manufacturer (none) -> Diodes Incorporated; PCBWay Sourcing Note (none) -> PCBWay turnkey; exact MPN; Power Rating (none) -> N/A; Sourcing URL (none) -> https://www.digikey.com/en/products/result?keywords=AP7343-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; Substitution Policy (none) -> NO SUBSTITUTE WITHOUT WRITTEN APPROVAL; Technology (none) -> Integrated circuit; Temperature Rating (none) -> -40..85 C minimum; Tolerance (none) -> N/A; Voltage Rating (none) -> Per datasheet
