File: fabrication/jlcpcb/source/hardware/Flight Controller.kicad_pcb (KiCad board)
At the start: 6 copper layers, 40.6 x 50.5 mm, 162 parts, among them J1 USB4110GFA, J10 CAN BUS, J11 MAVLINK SIGNAL-ONLY, J12 POWER1 REGULATED 5.2V IN, J2 FPV, J3 ST_LINK, J4 GPS, J5 Airspeed sensor, J6 OpenESC SIGNAL-ONLY, J7 RC Receiver, J8 VTX, J9 DJI, Q1 AO3407A, SW1 reset, SW2 MCU_BOOT, U1 TPS54302, U10 BMI270, U12 BMP388, U13 AT7456E, U14 SN65HVD230, U2 USBLC6-2SC6, U5 AP2112K-3.3, U6 AP7343-33W5-7, U7 STM32H743VITx, U8 ICM-42688-P, U9 W25Q128JVSIQ, Y1 ASE-8.000MHZ-LC-T, Y2 27Mhz 20pF

Commit message: docs: publish neutral engineering source, manufacturing and portfolio overview
Other:
- board text added: "FC V2"
- board text removed: "FC DRONE FC"
Changed lines of the file:
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@@
 		)
 	)
-	(gr_text "FC DRONE FC"
+	(gr_text "FC V2"
 		(at 128.699999 95.1 0)
 		(layer "B.SilkS")
