File: fabrication/jlcpcb/source/hardware/connectors.kicad_sch (KiCad schematic)
At the start: 53 parts, among them J10 CAN BUS, J11 MAVLINK SIGNAL-ONLY, J12 POWER1 REGULATED 5.2V IN, J2 FPV, J3 ST_LINK, J4 GPS, J5 Airspeed sensor, J6 OpenESC SIGNAL-ONLY, J7 RC Receiver, J8 VTX, J9 DJI

Commit message: docs: publish neutral engineering source, manufacturing and portfolio overview
Other:
- company: FC DRONE PROJECT -> Desan Vasu
- title: FC DRONE FC -> Flight Controller V2
Changed lines of the file:
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@@
 	(paper "User" 431.8 254)
 	(title_block
-		(title "FC DRONE FC")
+		(title "Flight Controller V2")
 		(date "2026-09-13")
 		(rev "A")
-		(company "FC DRONE PROJECT")
+		(company "Desan Vasu")
 		(comment 1 "Derived from upstream commit 0a60da1 under CERN-OHL-S-2.0")
 		(comment 2 "POWER/OPENESC REDESIGN IMPLEMENTED - BENCH VALIDATION REQUIRED")
