File: fabrication/pcbway/source/hardware/MCU.kicad_sch (KiCad schematic)
At the start: 33 parts, among them SW1 reset, SW2 MCU_BOOT, U7 STM32H743VIT6, Y1 ASE-8.000MHZ-L-C-T

Commit message: docs: publish neutral engineering source, manufacturing and portfolio overview
Other:
- company: FC DRONE PROJECT -> Desan Vasu
- title: FC DRONE FC -> Flight Controller V2
Changed lines of the file:
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@@
 	(paper "User" 457.2 279.4)
 	(title_block
-		(title "FC DRONE FC")
+		(title "Flight Controller V2")
 		(date "2026-09-13")
 		(rev "A")
-		(company "FC DRONE PROJECT")
+		(company "Desan Vasu")
 		(comment 1 "Derived from upstream commit 0a60da1 under CERN-OHL-S-2.0")
 		(comment 2 "POWER/OPENESC REDESIGN IMPLEMENTED - BENCH VALIDATION REQUIRED")
