File: fabrication/pcbway/source/hardware/Sensors.kicad_sch (KiCad schematic)
At the start: 43 parts, among them U10 BMI270, U11 LIS3MDLTR, U12 BMP388, U13 AT7456E, U14 SN65HVD230, U8 ICM-42688-P, U9 W25Q128JVSIQ, Y2 TSX-3225 27.00M-N0AANNG40RG3

Commit message: docs: publish neutral engineering source, manufacturing and portfolio overview
Other:
- company: FC DRONE PROJECT -> Desan Vasu
- title: FC DRONE FC -> Flight Controller V2
Changed lines of the file:
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@@
 	(paper "User" 635 279.4)
 	(title_block
-		(title "FC DRONE FC")
+		(title "Flight Controller V2")
 		(date "2026-09-13")
 		(rev "A")
-		(company "FC DRONE PROJECT")
+		(company "Desan Vasu")
 		(comment 1 "Derived from upstream commit 0a60da1 under CERN-OHL-S-2.0")
 		(comment 2 "POWER/OPENESC REDESIGN IMPLEMENTED - BENCH VALIDATION REQUIRED")
