File: fabrication/pcbway/source/hardware/power.kicad_sch (KiCad schematic)
At the start: 44 parts, among them J1 USB4110GFA, Q1 AO3407A, U1 TPS54302, U2 USBLC6-2SC6, U3 INA226, U5 AP2112K-3.3, U6 AP7343-33W5-7

Commit message: docs: publish neutral engineering source, manufacturing and portfolio overview
Other:
- company: FC DRONE PROJECT -> Desan Vasu
- title: FC DRONE FC -> Flight Controller V2
Changed lines of the file:
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@@
 	(paper "User" 584.2 279.4)
 	(title_block
-		(title "FC DRONE FC")
+		(title "Flight Controller V2")
 		(date "2026-09-13")
 		(rev "A")
-		(company "FC DRONE PROJECT")
+		(company "Desan Vasu")
 		(comment 1 "Derived from upstream commit 0a60da1 under CERN-OHL-S-2.0")
 		(comment 2 "POWER/OPENESC REDESIGN IMPLEMENTED - BENCH VALIDATION REQUIRED")
